File: mini_module_template/mini_module_template.kicad_pcb (KiCad board)
At the start: 4 copper layers, 100 x 60 mm, 150 parts, among them IC1 TJA1044GTK_3Z, IC2 TJA1044GTK_3Z, IC3 LMR16030SDDAR, J1 SWD, J2 Conn_01x02, J4 USB_C_Receptacle_USB2.0, J6 Conn_01x02, J7 RJ45_LED_Shielded, J8 RJ45_LED_Shielded, Q1 S9013, SW2 NRST, SW5 SW_DIP_x02, U1 CH334R, U2 FM24CL16B, U3 STM32F103CB, U4 AZ1117-3.3, U6 IP4220CZ6, U8 TS3USB30EDGSR, U9 STM32F446RETx, Y1 8MHz, Y2 8MHz, Y3 32.768kHz, Y4 12Mhz

Commit message: final check rev A
Parts:
- C55: footprint Capacitor_SMD:C_0603_1608Metric -> Capacitor_SMD:C_0402_1005Metric
- R27: value 430k -> 43k; footprint Resistor_SMD:R_0603_1608Metric -> Resistor_SMD:R_0402_1005Metric
- R29: value 1k -> 220
- R30: value 10k -> 1k; footprint Resistor_SMD:R_0603_1608Metric -> Resistor_SMD:R_0402_1005Metric
- moved C12 5.06 mm to (103.3, 85.8), turned to 135 degrees
- moved C11 4.76 mm to (101.9, 84.4), turned to -45 degrees
- moved C56 3.66 mm to (101.2, 80.2), turned to -90 degrees
- moved R2 3.25 mm to (106.1, 87.4), turned to -45 degrees
- moved C57 2.67 mm to (101.2, 82.1), turned to 90 degrees
- moved C9 1.77 mm to (105.4, 88.1), turned to 135 degrees
- moved R27 1.05 mm to (103.8, 90.5)
- moved Y1 0.94 mm to (101.0, 86.7), turned to 135 degrees
- moved Y3 0.37 mm to (99.5, 81.1)
Routing:
- net GND: track 119.0 -> 122.7 mm, vias 113 -> 116
- net Net-(U9-PH1): track 11.1 -> 7.45 mm
- net Net-(U9-PC14): track 9.93 -> 7.07 mm
- net /MCU/NRST: track 111.8 -> 110.1 mm
- net VCC: track 14.5 -> 15.8 mm
- net Net-(U9-PC15): track 8.82 -> 7.51 mm
- net Net-(U9-PH0): track 11.1 -> 10.1 mm
- net /CAN/CAN1+: track 140.7 -> 140.0 mm
- net /MCU/V_SENSE: track 10.9 -> 11.5 mm
- net /CAN/CAN1-: track 122.7 -> 122.2 mm

Commit message: fixed issue woth oncvorrect usb pin
Connections:
- J7 pad 7: /CAN/USB_UPSTREAM_D+ -> /CAN/USB_UPSTREAM_D-
- J7 pad 8: /CAN/USB_UPSTREAM_D- -> /CAN/USB_UPSTREAM_D+
Routing:
- net /CAN/USB_UPSTREAM_D-: track 44.1 -> 40.6 mm, vias 2 -> 1
- net /CAN/USB_UPSTREAM_D+: track 41.5 -> 42.4 mm, vias 2 -> 1
- net GND: vias 116 -> 113
Changed lines of the file:
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@@
 			(layers "*.Cu" "*.Mask")
 			(remove_unused_layers no)
-			(net 133 "/CAN/USB_UPSTREAM_D+")
+			(net 131 "/CAN/USB_UPSTREAM_D-")
 			(pintype "passive")
 		)
@@
 			(layers "*.Cu" "*.Mask")
 			(remove_unused_layers no)
-			(net 131 "/CAN/USB_UPSTREAM_D-")
+			(net 133 "/CAN/USB_UPSTREAM_D+")
 			(pintype "passive")
 		)
@@
 	)
 	(via
-		(at 177.6 89)
-		(size 0.55)
-		(drill 0.35)
-		(layers "F.Cu" "B.Cu")
-		(net 2)
-	)
-	(via
 		(at 114.5 67.6)
 		(size 0.55)
@@
 	)
 	(via
-		(at 179 88.4)
-		(size 0.55)
-		(drill 0.35)
-		(layers "F.Cu" "B.Cu")
-		(net 2)
-	)
-	(via
 		(at 127.98 62.52)
 		(size 0.55)
@@
 	)
 	(via
-		(at 178.425 86.934862)
-		(size 0.55)
-		(drill 0.35)
-		(layers "F.Cu" "B.Cu")
-		(net 2)
-	)
-	(via
 		(at 162 63)
 		(size 0.6)
@@
 	)
 	(segment
-		(start 178.2 88.4)
-		(end 178.103064 88.303064)
-		(width 0.3)
-		(layer "F.Cu")
-		(net 131)
-	)
-	(segment
 		(start 159.07 68.219999)
 		(end 160.007644 68.219999)
@@
 	)
 	(segment
-		(start 178.103064 88.303064)
-		(end 175.396936 88.303064)
-		(width 0.3)
-		(layer "F.Cu")
-		(net 131)
-	)
-	(segment
 		(start 161.3 69.9)
 		(end 161.3 70.149997)
@@
 	)
 	(segment
-		(start 175.396936 88.303064)
-		(end 173 90.7)
-		(width 0.3)
-		(layer "F.Cu")
-		(net 131)
-	)
-	(segment
 		(start 161.3 69.512355)
 		(end 161.3 69.9)
@@
 		(net 131)
 	)
-	(segment
-		(start 170.218001 90.7)
-		(end 169.68 90.161999)
-		(width 0.3)
-		(layer "F.Cu")
-		(net 131)
-	)
-	(segment
-		(start 173 90.7)
-		(end 170.218001 90.7)
-		(width 0.3)
-		(layer "F.Cu")
-		(net 131)
-	)
-	(via
-		(at 178.2 88.4)
-		(size 0.55)
-		(drill 0.35)
-		(layers "F.Cu" "B.Cu")
-		(net 131)
-	)
 	(via
 		(at 161.149997 70.3)
@@
 	)
 	(segment
-		(start 161.224998 73.224998)
-		(end 161.224998 70.375001)
+		(start 177.2 88.895734)
+		(end 177.2 79.7)
 		(width 0.3)
 		(layer "B.Cu")
@@
 	)
 	(segment
-		(start 174.8 77.3)
-		(end 171.8 77.3)
+		(start 161.224998 70.375001)
+		(end 161.149997 70.3)
 		(width 0.3)
 		(layer "B.Cu")
@@
 	)
 	(segment
-		(start 177.2 87.449117)
-		(end 177.2 79.7)
+		(start 171.46 89.146)
+		(end 171.875998 89.561998)
 		(width 0.3)
 		(layer "B.Cu")
@@
 	)
 	(segment
-		(start 177.2 79.7)
-		(end 174.8 77.3)
+		(start 163.095 75.095)
+		(end 161.224998 73.224998)
 		(width 0.3)
 		(layer "B.Cu")
@@
 	)
 	(segment
-		(start 178.150883 88.4)
-		(end 177.2 87.449117)
+		(start 176.533736 89.561998)
+		(end 176.847867 89.247867)
 		(width 0.3)
 		(layer "B.Cu")
@@
 	)
 	(segment
-		(start 161.224998 70.375001)
-		(end 161.149997 70.3)
+		(start 177.2 79.7)
+		(end 174.8 77.3)
 		(width 0.3)
 		(layer "B.Cu")
@@
 	)
 	(segment
-		(start 163.095 75.095)
-		(end 161.224998 73.224998)
+		(start 174.8 77.3)
+		(end 171.8 77.3)
 		(width 0.3)
 		(layer "B.Cu")
@@
 	)
 	(segment
-		(start 169.595 75.095)
-		(end 163.095 75.095)
+		(start 161.224998 73.224998)
+		(end 161.224998 70.375001)
+		(width 0.3)
+		(layer "B.Cu")
+		(net 131)
+	)
+	(segment
+		(start 171.875998 89.561998)
+		(end 176.533736 89.561998)
 		(width 0.3)
 		(layer "B.Cu")
@@
 	)
 	(segment
-		(start 178.2 88.4)
-		(end 178.150883 88.4)
+		(start 176.847867 89.247867)
+		(end 177.2 88.895734)
+		(width 0.3)
+		(layer "B.Cu")
+		(net 131)
+	)
+	(segment
+		(start 169.595 75.095)
+		(end 163.095 75.095)
 		(width 0.3)
 		(layer "B.Cu")
@@
 	)
 	(segment
-		(start 171.46 89.76)
-		(end 171.46 89.146)
-		(width 0.3)
-		(layer "F.Cu")
-		(net 133)
-	)
-	(segment
 		(start 161.9 69.494407)
 		(end 161.9 69.9)
@@
 	)
 	(segment
-		(start 178.479253 87.703063)
-		(end 175.196937 87.703063)
-		(width 0.3)
-		(layer "F.Cu")
-		(net 133)
-	)
-	(segment
-		(start 172.8 90.1)
-		(end 171.8 90.1)
-		(width 0.3)
-		(layer "F.Cu")
-		(net 133)
-	)
-	(segment
-		(start 175.196937 87.703063)
-		(end 172.8 90.1)
-		(width 0.3)
-		(layer "F.Cu")
-		(net 133)
-	)
-	(segment
 		(start 161.9 69.9)
 		(end 161.9 70.3)
@@
 		(net 133)
 	)
-	(segment
-		(start 171.8 90.1)
-		(end 171.46 89.76)
-		(width 0.3)
-		(layer "F.Cu")
-		(net 133)
-	)
 	(via
 		(at 161.9 70.3)
@@
 		(net 133)
 	)
-	(via
-		(at 178.479253 87.703063)
-		(size 0.55)
-		(drill 0.35)
-		(layers "F.Cu" "B.Cu")
-		(net 133)
-	)
 	(segment
-		(start 161.824999 73.117893)
-		(end 163.202126 74.49502)
+		(start 177.8 79.5)
+		(end 175.1 76.8)
 		(width 0.3)
 		(layer "B.Cu")
@@
 	)
 	(segment
-		(start 161.9 70.3)
-		(end 161.824999 70.375001)
+		(start 161.824999 70.375001)
+		(end 161.9 70.3)
 		(width 0.3)
 		(layer "B.Cu")
@@
 	)
 	(segment
-		(start 177.8 87.200587)
-		(end 178.302476 87.703063)
+		(start 175.1 76.8)
+		(end 172.037918 76.8)
 		(width 0.3)
 		(layer "B.Cu")
@@
 	(segment
 		(start 169.732938 74.49502)
-		(end 172.037918 76.8)
+		(end 163.202126 74.49502)
 		(width 0.3)
 		(layer "B.Cu")
@@
 	)
 	(segment
-		(start 177.8 79.5)
-		(end 177.8 87.200587)
+		(start 171.885398 90.173)
+		(end 171.896399 90.161999)
 		(width 0.3)
 		(layer "B.Cu")
@@
 	)
 	(segment
-		(start 178.302476 87.703063)
-		(end 178.479253 87.703063)
+		(start 171.034602 90.173)
+		(end 171.885398 90.173)
 		(width 0.3)
 		(layer "B.Cu")
@@
 	)
 	(segment
-		(start 172.037918 76.8)
-		(end 175.1 76.8)
+		(start 163.202126 74.49502)
+		(end 161.824999 73.117893)
 		(width 0.3)
 		(layer "B.Cu")
@@
 	)
 	(segment
-		(start 175.1 76.8)
+		(start 177.8 89.144266)
 		(end 177.8 79.5)
 		(width 0.3)
@@
 	)
 	(segment
-		(start 163.202126 74.49502)
+		(start 172.037918 76.8)
 		(end 169.732938 74.49502)
 		(width 0.3)
@@
 	)
 	(segment
-		(start 161.824999 70.375001)
-		(end 161.824999 73.117893)
+		(start 176.782267 90.161999)
+		(end 177.8 89.144266)
+		(width 0.3)
+		(layer "B.Cu")
+		(net 133)
+	)
+	(segment
+		(start 171.023601 90.161999)
+		(end 171.034602 90.173)
+		(width 0.3)
+		(layer "B.Cu")
+		(net 133)
+	)
+	(segment
+		(start 161.824999 73.117893)
+		(end 161.824999 70.375001)
+		(width 0.3)
+		(layer "B.Cu")
+		(net 133)
+	)
+	(segment
+		(start 169.68 90.161999)
+		(end 171.023601 90.161999)
+		(width 0.3)
+		(layer "B.Cu")
+		(net 133)
+	)
+	(segment
+		(start 171.896399 90.161999)
+		(end 176.782267 90.161999)
 		(width 0.3)
 		(layer "B.Cu")

Commit message: final rev
Routing:
- net /MCU/USR_LED2: track 16.8 -> 18.8 mm
- net /MCU/NRST: track 110.1 -> 109.0 mm
Changed lines of the file:
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@@
 	)
 	(segment
-		(start 101.218553 79.68005)
-		(end 101.226371 79.687868)
-		(width 0.254)
-		(layer "F.Cu")
-		(net 2)
-	)
-	(segment
 		(start 143.9 60.775)
 		(end 144.66 61.535)
@@
 	)
 	(segment
-		(start 101.226371 79.687868)
-		(end 101.99637 79.687868)
-		(width 0.254)
-		(layer "F.Cu")
-		(net 2)
-	)
-	(segment
 		(start 135.5 63.6)
 		(end 134.909999 63.6)
@@
 	)
 	(segment
+		(start 100.841441 79.178023)
+		(end 101.218553 79.555135)
+		(width 0.254)
+		(layer "F.Cu")
+		(net 2)
+	)
+	(segment
 		(start 102.9 78.971178)
 		(end 103.370589 78.500589)
@@
 	)
 	(segment
+		(start 101.218553 79.555135)
+		(end 101.218553 79.68005)
+		(width 0.254)
+		(layer "F.Cu")
+		(net 2)
+	)
+	(segment
 		(start 99.3725 62.662499)
 		(end 98.862499 62.662499)
@@
 	)
 	(via
-		(at 101.99637 79.687868)
+		(at 100.841441 79.178023)
 		(size 0.55)
 		(drill 0.35)
@@
 	)
 	(segment
-		(start 107.954763 79.964763)
-		(end 107.77 79.78)
-		(width 0.254)
-		(layer "F.Cu")
-		(net 3)
-	)
-	(segment
 		(start 139.439998 76.41)
 		(end 125.81 76.41)
@@
 	)
 	(segment
-		(start 107.356839 81.682501)
-		(end 107.954763 81.084577)
-		(width 0.254)
-		(layer "F.Cu")
-		(net 3)
-	)
-	(segment
 		(start 105.732306 88.446518)
 		(end 105.77473 88.446518)
@@
 	)
 	(segment
-		(start 102.800224 76.2)
-		(end 102.8 76.2)
-		(width 0.3)
-		(layer "F.Cu")
-		(net 23)
-	)
-	(segment
-		(start 102.8 75.751358)
-		(end 103.025679 75.525679)
-		(width 0.3)
-		(layer "F.Cu")
-		(net 23)
-	)
-	(segment
-		(start 102.8 76.2)
-		(end 102.8 75.751358)
-		(width 0.3)
-		(layer "F.Cu")
-		(net 23)
-	)
-	(segment
-		(start 104.800224 78.2)
-		(end 102.800224 76.2)
-		(width 0.3)
-		(layer "F.Cu")
-		(net 23)
-	)
-	(segment
-		(start 106.4 78.8)
-		(end 105.8 78.2)
-		(width 0.3)
+		(start 103.165658 80.485658)
+		(end 101.62 78.94)
+		(width 0.2)
 		(layer "F.Cu")
 		(net 23)
 	)
 	(segment
-		(start 105.8 78.2)
-		(end 104.800224 78.2)
-		(width 0.3)
+		(start 105.018148 80.485658)
+		(end 103.165658 80.485658)
+		(width 0.2)
 		(layer "F.Cu")
 		(net 23)
@@
 	(segment
 		(start 105.589072 79.914734)
-		(end 106.4 79.103806)
-		(width 0.3)
+		(end 105.018148 80.485658)
+		(width 0.2)
 		(layer "F.Cu")
 		(net 23)
 	)
 	(segment
-		(start 106.4 79.103806)
-		(end 106.4 78.8)
-		(width 0.3)
+		(start 101.62 78.94)
+		(end 101.62 76.78)
+		(width 0.2)
 		(layer "F.Cu")
 		(net 23)
 	)
 	(via
-		(at 103.025679 75.525679)
+		(at 101.62 76.78)
 		(size 0.55)
 		(drill 0.35)
@@
 	)
 	(segment
-		(start 104.365 69.725)
-		(end 104.88 69.21)
+		(start 103.625 70.465)
+		(end 104.66 69.43)
 		(width 0.3)
 		(layer "B.Cu")
@@
 	)
 	(segment
-		(start 103.025679 75.525679)
-		(end 103.625 74.926358)
+		(start 104.365 69.725)
+		(end 104.88 69.21)
 		(width 0.3)
 		(layer "B.Cu")
@@
 	)
 	(segment
-		(start 103.625 70.465)
-		(end 104.66 69.43)
+		(start 101.62 76.78)
+		(end 103.625 74.775)
 		(width 0.3)
 		(layer "B.Cu")
@@
 	)
 	(segment
-		(start 103.625 74.926358)
+		(start 103.625 74.775)
 		(end 103.625 70.465)
 		(width 0.3)
@@
 	)
 	(segment
-		(start 101.444714 80.866211)
-		(end 101.218553 80.64005)
-		(width 0.254)
-		(layer "F.Cu")
-		(net 143)
-	)
-	(segment
 		(start 100.478503 79.9)
 		(end 101.218553 80.640049)
@@
 	)
 	(segment
-		(start 105.942625 80.268287)
-		(end 105.344701 80.866211)
+		(start 101.718503 81.14)
+		(end 101.218553 80.64005)
 		(width 0.254)
 		(layer "F.Cu")
@@
 	)
 	(segment
-		(start 105.344701 80.866211)
-		(end 101.444714 80.866211)
+		(start 105.942625 80.268287)
+		(end 105.070912 81.14)
 		(width 0.254)
 		(layer "F.Cu")
@@
 		(layer "F.Cu")
 		(net 143)
+	)
+	(segment
+		(start 105.070912 81.14)
+		(end 101.718503 81.14)
+		(width 0.254)
+		(layer "F.Cu")
+		(net 143)
