File: PCB-source/CAN_TR.kicad_sch (KiCad schematic)
At the start: 4 parts, among them U500 TJA1044GTK_3Z

Commit message: Finish component and diffpair placement
Other:
- title: MMS2 -> CAN transceiver
Changed lines of the file:
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@@
 	(paper "A4")
 	(title_block
-		(title "MMS2")
+		(title "CAN transceiver")
 		(date "2025-04-22")
 		(rev "A")
