File: PCB-source/QSPI_FLASH.kicad_sch (KiCad schematic)
At the start: 2 parts, among them U100 W25Q128

Commit message: Finish component and diffpair placement
Other:
- title: MMS2 -> QSPI flash
Changed lines of the file:
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@@
 	(paper "A4")
 	(title_block
-		(title "MMS2")
+		(title "QSPI flash")
 		(date "2025-04-22")
 		(rev "A")
