File: PCB-source/USB switch.kicad_sch (KiCad schematic)
At the start: 5 parts, among them U801 FSUSB42UMX

Commit message: Finish component and diffpair placement
Parts:
- U801: footprint kicad-footprints:UFQFN-10_1.4x1.8 -> UFQFN-10_1.4x1.8:UFQFN-10_1.4x1.8
Other:
- title: MMS2 -> USB Switch
Changed lines of the file:
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@@
 	(paper "A4")
 	(title_block
-		(title "MMS2")
+		(title "USB Switch")
 		(date "2025-04-22")
 		(rev "A")
@@
 			)
 		)
-		(property "Footprint" "kicad-footprints:UFQFN-10_1.4x1.8"
+		(property "Footprint" "UFQFN-10_1.4x1.8:UFQFN-10_1.4x1.8"
 			(at 135.89 68.834 0)
 			(effects
