File: PCB-source/USBC_CONN.kicad_sch (KiCad schematic)
At the start: 7 parts, among them J800 USB_C_Receptacle_USB2.0_16P, U401 TPD2E2U06DCK

Commit message: vrm VIP
Changed lines of the file:
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@@
+	)
+	(junction
+		(at 165.1 72.39)
+		(diameter 0)
+		(color 0 0 0 0)
 	)
 	(junction
@@
 	(wire
 		(pts
+			(xy 165.1 72.39) (xy 181.61 72.39)
+		)
+		(stroke
+			(width 0)
+			(type default)
+		)
+	)
+	(wire
+		(pts
 			(xy 101.6 127) (xy 101.6 128.27)
 		)
@@
 	(wire
 		(pts
-			(xy 139.7 72.39) (xy 181.61 72.39)
+			(xy 139.7 72.39) (xy 165.1 72.39)
 		)
 		(stroke
@@
 		(pts
 			(xy 93.98 127) (xy 93.98 128.27)
+		)
+		(stroke
+			(width 0)
+			(type default)
+		)
+	)
+	(wire
+		(pts
+			(xy 165.1 69.85) (xy 165.1 72.39)
 		)
 		(stroke
@@
 					(unit 1)
 				)
+			)
+		)
+	)
+	(symbol
+		(lib_id "power:VBUS")
+		(at 165.1 69.85 0)
+		(unit 1)
+		(exclude_from_sim no)
+		(in_bom yes)
+		(on_board yes)
+		(dnp no)
+		(fields_autoplaced yes)
+		(property "Reference" "#PWR018"
+			(at 165.1 73.66 0)
+			(effects
+				(font
+					(size 1.27 1.27)
+				)
+				(hide yes)
+			)
+		)
+		(property "Value" "VBUS"
+			(at 165.1 64.77 0)
+			(effects
+				(font
+					(size 1.27 1.27)
+				)
+			)
+		)
+		(property "Footprint" ""
+			(at 165.1 69.85 0)
+			(effects
+				(font
+					(size 1.27 1.27)
+				)
+				(hide yes)
+			)
+		)
+		(property "Datasheet" ""
+			(at 165.1 69.85 0)
+			(effects
+				(font
+					(size 1.27 1.27)
+				)
+				(hide yes)
+			)
+		)
+		(property "Description" "Power symbol creates a global label with name \"VBUS\""
+			(at 165.1 69.85 0)
+			(effects
+				(font
+					(size 1.27 1.27)
+				)
+				(hide yes)
+			)
+		)
+		(pin "1"
+		)
+		(instances
+			(project "MMS2"
+				(path "/6596548a-44e0-46d8-8624-fd71cf4a3e17/9171ecef-cf73-4f55-b1f0-c4c88f6b0a62"
+					(reference "#PWR018")
+					(unit 1)
+				)

Commit message: Finish component and diffpair placement
Parts:
- U401: value TPD2E2U06DCK -> TPD2EUSB30DRTR-TP; footprint Package_TO_SOT_SMD:SOT-323_SC-70 -> Package_TO_SOT_SMD:SOT-723; LCSC (none) -> C2844720
Other:
- title: MMS2 -> USB-C
Changed lines of the file:
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@@
 	(paper "A4")
 	(title_block
-		(title "MMS2")
+		(title "USB-C")
 		(date "2025-04-22")
 		(rev "A")
@@
 			)
 		)
-		(property "Value" "TPD2E2U06DCK"
+		(property "Value" "TPD2EUSB30DRTR-TP"
 			(at 158.75 101.5999 0)
 			(effects
@@
 			)
 		)
-		(property "Footprint" "Package_TO_SOT_SMD:SOT-323_SC-70"
+		(property "Footprint" "Package_TO_SOT_SMD:SOT-723"
 			(at 134.62 106.68 0)
 			(effects
@@
 			)
 		)
-		(property "Datasheet" "http://www.ti.com/lit/ds/symlink/tpd2e2u06.pdf"
+		(property "Datasheet" "https://www.lcsc.com/datasheet/C2844720.pdf"
 			(at 149.86 95.25 0)
 			(effects
@@
 			(at 154.94 100.33 0)
 			(effects
+				(font
+					(size 1.27 1.27)
+				)
+				(hide yes)
+			)
+		)
+		(property "LCSC" "C2844720"
+			(at 154.94 100.33 0)
+			(effects
