File: PCB-source/LMR36520ADDAR.kicad_sch (KiCad schematic)
At the start: 27 parts, among them U2 LMR36520ADDAR

Commit message: in progress
Parts:
- removed C21: 22uF, PCM_JLCPCB:C_0805, symbol PCM_JLCPCB-Capacitors:0805,22uF
- removed D1: ESDBL18VD3N, Diode_SMD:D_SOD-323, symbol PCM_JLCPCB-Diodes:TVS-Bi,SMAJ40CA
- removed R8, R9: 100kΩ, PCM_JLCPCB:R_0402, symbol PCM_JLCPCB-Resistors:0402,100kΩ
- added C21, C27: 1uF, PCM_JLCPCB:C_0402, symbol PCM_JLCPCB-Capacitors:0402,1uF
- added C23, C24, C25, C28: 22uF, PCM_JLCPCB:C_0805, symbol PCM_JLCPCB-Capacitors:0805,22uF
- added D1: SMF58CA, PCM_JLCPCB:D_SOD-123FL, symbol PCM_JLCPCB-Diodes:TVS-Uni,SMF58CA
- added R8, R9: 24.9kΩ, PCM_JLCPCB:R_0402, symbol PCM_JLCPCB-Resistors:0402,24kΩ
Connections:
- net GND: now also C21.2, C23.2, C24.2, C25.2, C27.2, C28.2, D1.2, R9.2
- net Vin: now also R8.1
- net Vout: now also C21.1, C23.1, C24.1, C25.1, C27.1, C28.1
- net Cap_protec: now reaches C1.2, C14.2, C15.1, C2.1, C4.2, C5.1, C6.2, C7.1, C8.2, C9.1
- net Cap_protec: now also D1.1, R8.2, R9.1
Other:
- note added: "IEC 60664-1 Material Group III (CTI < 400; typical FR-4 = IIIa): 1.25 mm"
- note added: "INFORMATION"
- note added: "KEEP CRIPPAGE DISTANCE 1.26MM MIN!"
- moved on the sheet: C1, C10, C14, C15, C16, C2, C4, C5, C6, C7, C8, C9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
