File: PCB-source/MMS2.kicad_pcb (KiCad board)
At the start: 2 copper layers, 90 x 50 mm, 178 parts, among them J1 86093488324755V1LF, J6 AMASS XT60, J7 AMASS XT60, J8 RJ45_LED_Shielded, J800 USB_C_Receptacle_USB2.0_16P, J9 RJ45_LED_Shielded, Q2 AO3400A, Q3 AO3400A, Q5 AO3400A, Q6 AO3400A, Q7 AO3400A, Q700 MMST3904, SW5 SW_DIP_x02, U1 STM32H563VGTx, U100 W25Q128, U2 LMR36520ADDAR, U3 TPD2EUSB30DRTR-TP, U301 TPS563200, U302 CH334P, U4 TPD2EUSB30DRTR-TP, U401 TPD2EUSB30DRTR-TP, U5 LM74700, U500 TJA1044GTK_3Z, U501 TJA1044GTK_3Z, U700 STM32F103CBTx, U801 FSUSB42UMX, X300 Q13FC1350000400, Y400 ASE-xxxMHz, Y700 Crystal_GND24, Y900 Crystal_GND24

Commit message: pinout start
Parts:
- removed TP302: TestPoint, TestPoint:TestPoint_Pad_D1.0mm
- moved D301 32.4 mm to (104.8, 110.7), turned to 0 degrees
- moved R401 27.8 mm to (119.4, 85.5), turned to 0 degrees
- moved C410 25.9 mm to (117.4, 85.5)
- moved R805 24.8 mm to (88.9, 100.6), turned to 0 degrees
- moved R402 23.6 mm to (121.7, 85.5), turned to 0 degrees
- moved C434 19.7 mm to (123.6, 85.0), turned to -90 degrees
- moved TP706 18.8 mm to (109.8, 81.2)
- moved TP700 18.8 mm to (105.7, 83.2)
- moved TP701 18.8 mm to (107.8, 83.2)
- moved TP702 18.8 mm to (109.8, 83.2)
- moved TP704 18.8 mm to (105.7, 81.2)
- moved TP705 18.8 mm to (107.7, 81.2)
- moved TP703 18.8 mm to (111.9, 83.2)
- moved R800 17.5 mm to (88.9, 96.6), turned to 0 degrees
- moved R804 16.7 mm to (102.4, 108.8), turned to 90 degrees
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Connections:
- C17 pad 1: /VRM/TPS563201/SW_3V3 -> /VRM/TPS563201/+3V3_UNPROTEC
- JP301 pad 2: /VRM/TPS563201/VOUT -> /VRM/TPS563201/+3V3_UNPROTEC
- L301 pad 1: /VRM/TPS563201/SW_3V3 -> /VRM/TPS563201/+3V3_UNPROTEC
- U301 pad 2: /VRM/TPS563201/SW_3V3 -> /VRM/TPS563201/+3V3_UNPROTEC
Routing:
- net /CAN auto terminator/CAN2.+: track 17.8 -> 46.3 mm
- net /USB switch/USBC_CONN.D+: track 4.16 -> 31.7 mm, vias 0 -> 2
- net /USB switch/USBC_CONN.D-: track 5.09 -> 32.5 mm, vias 0 -> 2
- net /CAN auto terminator/CAN1.+: track 17.0 -> 32.8 mm, vias 0 -> 1
- net /CAN auto terminator/CAN2.-: track 22.0 -> 37.5 mm
- net /CAN auto terminator/CAN1.-: track 15.8 -> 26.5 mm, vias 0 -> 1
- net +3V3: track 4.71 -> 14.3 mm
- net Net-(C46-Pad1): track 0.00 -> 9.59 mm
- net VBUS: track 14.3 -> 6.53 mm
- net Net-(U302-XI): track 0.00 -> 6.57 mm
- net Net-(Q700-B): track 0.00 -> 4.85 mm
- net +5V: track 1.16 -> 5.86 mm, vias 0 -> 1
- net /MMS_CONNECTOR_UPSTREAM/USB_MMS_CONN.D-: track 17.7 -> 13.3 mm
- net /CAN_TR1/CAN.TX: track 0.00 -> 4.27 mm, vias 0 -> 1
- net Net-(U302-XO): track 0.00 -> 4.16 mm
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Other:
- board text added: "(c) 2025"
- board text added: "2"
- board text added: "ChainBus"
- board text added: "Designed with by Artem.H"
- board text added: "MINI MODULAR SYSTEM"
- board text added: "connector powered by"
- board text removed: "Connector powered by ChainBus"

Commit message: in progress
Parts:
- removed C21: 22uF, PCM_JLCPCB:C_0805
- removed J6: AMASS XT60, Connector_AMASS:AMASS_XT60PW-M_1x02_P7.20mm_Horizontal
- added C23: 22uF, PCM_JLCPCB:C_0805, F.Cu at (129.7, 134.4)
- added C24: 22uF, PCM_JLCPCB:C_0805, F.Cu at (127.7, 134.4)
- added C25: 22uF, PCM_JLCPCB:C_0805, F.Cu at (125.7, 134.4)
- added C27: 1uF, PCM_JLCPCB:C_0402, F.Cu at (112.6, 135.7)
- added C28: 22uF, PCM_JLCPCB:C_0805, F.Cu at (131.7, 130.4)
- added H1: M3 mount, MountingHole:MountingHole_3.2mm_M3_DIN965_Pad, F.Cu at (3.08, 3.08)
- added H2: M3 mount, MountingHole:MountingHole_3.2mm_M3_DIN965_Pad, F.Cu at (151.1, 107.0)
- added H3: M3 mount, MountingHole:MountingHole_3.2mm_M3_DIN965_Pad, F.Cu at (3.08, 10.2)
- added H4: M3 mount, MountingHole:MountingHole_3.2mm_M3_DIN965_Pad, F.Cu at (164.0, 129.0)
- added H4: M3 mount, MountingHole:MountingHole_3.2mm_M3_DIN965_Pad, F.Cu at (94.0, 92.0)
- added H4: M3 mount, MountingHole:MountingHole_3.2mm_M3_DIN965_Pad, F.Cu at (86.0, 129.0)
- added J2: AMASS XT60, XT60:AMASS_XT60PW-M_1x02_P7.20mm_Horizontal, F.Cu at (94.5, 132.9)
- added TP302: TestPoint, TestPoint:TestPoint_Pad_D1.0mm, F.Cu at (108.3, 80.5)
- D1: value ESDBL18VD3N -> SMF58CA; footprint Diode_SMD:D_SOD-323 -> PCM_JLCPCB:D_SOD-123FL
- J7: footprint Connector_AMASS:AMASS_XT60PW-M_1x02_P7.20mm_Horizontal -> XT60:AMASS_XT60PW-F_1x02_P7.20mm_Horizontal
- R8, R9: value 100kΩ -> 24.9kΩ
- moved R400 80.1 mm to (102.6, 83.5), turned to 0 degrees
- moved R404 80.1 mm to (104.5, 81.6)
- moved R403 76.9 mm to (106.4, 84.5), turned to 0 degrees
- moved C416 75.9 mm to (104.5, 84.5), turned to 0 degrees
- moved R405 75.9 mm to (102.6, 84.5), turned to 0 degrees
- moved R407 75.8 mm to (108.4, 83.5), turned to 0 degrees
- moved C415 75.5 mm to (104.5, 83.5), turned to 0 degrees
- moved R408 73.6 mm to (108.4, 84.5), turned to 0 degrees
- moved R406 71.2 mm to (108.4, 82.5)
- moved J7 60.4 mm to (156.5, 133.0), turned to -90 degrees
- moved R409 30.0 mm to (102.6, 82.5), turned to 0 degrees
- moved C700 24.8 mm to (102.0, 67.4), turned to 0 degrees
- moved C45 24.7 mm to (91.2, 99.4), turned to 90 degrees
- moved R703 24.3 mm to (102.0, 69.2)
- moved R51 23.9 mm to (89.6, 99.8)
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Connections:
- C1 pad 1: /VRM/LMR36520ADDAR/LMR36520ADDAR_VIN -> BRD_VIN
- C1 pad 2: Net-(C1-Pad2) -> /VRM/LMR36520ADDAR/Cap_protec
- C14 pad 1: /VRM/LMR36520ADDAR/LMR36520ADDAR_VIN -> BRD_VIN
- C14 pad 2: Net-(C1-Pad2) -> /VRM/LMR36520ADDAR/Cap_protec
- C15 pad 1: Net-(C1-Pad2) -> /VRM/LMR36520ADDAR/Cap_protec
- C17 pad 1: /VRM/TPS563201/+3V3_UNPROTEC -> /VRM/TPS563201/SW_3V3
- C2 pad 1: Net-(C1-Pad2) -> /VRM/LMR36520ADDAR/Cap_protec
- C4 pad 1: /VRM/LMR36520ADDAR/LMR36520ADDAR_VIN -> BRD_VIN
- C4 pad 2: Net-(C1-Pad2) -> /VRM/LMR36520ADDAR/Cap_protec
- C5 pad 1: Net-(C1-Pad2) -> /VRM/LMR36520ADDAR/Cap_protec
- C6 pad 1: /VRM/LMR36520ADDAR/LMR36520ADDAR_VIN -> BRD_VIN
- C6 pad 2: Net-(C1-Pad2) -> /VRM/LMR36520ADDAR/Cap_protec
- C7 pad 1: Net-(C1-Pad2) -> /VRM/LMR36520ADDAR/Cap_protec
- C8 pad 1: /VRM/LMR36520ADDAR/LMR36520ADDAR_VIN -> BRD_VIN
- C8 pad 2: Net-(C1-Pad2) -> /VRM/LMR36520ADDAR/Cap_protec
- C9 pad 1: Net-(C1-Pad2) -> /VRM/LMR36520ADDAR/Cap_protec
- D1 pad 1: GND -> /VRM/LMR36520ADDAR/Cap_protec
- D1 pad 2: Net-(C1-Pad2) -> GND
- J1 pad A1: unconnected-(J1-PadA1) -> /Interboard_connector/I2C1.SDA
- J1 pad A10: unconnected-(J1-PadA10) -> /Interboard_connector/UART_ADDR.2
- J1 pad A11: unconnected-(J1-PadA11) -> /Interboard_connector/SPI.MISO
- J1 pad A12: unconnected-(J1-PadA12) -> /Interboard_connector/SPI.MOSI
- J1 pad A13: unconnected-(J1-PadA13) -> /Interboard_connector/SPI.CK
- J1 pad A14: unconnected-(J1-PadA14) -> /Interboard_connector/SPI_ADDR.0
- J1 pad A15: unconnected-(J1-PadA15) -> /Interboard_connector/SPI_ADDR.1
- J1 pad A16: unconnected-(J1-PadA16) -> /Interboard_connector/SPI_ADDR.2
- J1 pad A2: unconnected-(J1-PadA2) -> /Interboard_connector/I2C1.SCL
- J1 pad A3: unconnected-(J1-PadA3) -> /Interboard_connector/I2C_ADDR.0
- J1 pad A4: unconnected-(J1-PadA4) -> /Interboard_connector/I2C_ADDR.1
- J1 pad A5: unconnected-(J1-PadA5) -> /Interboard_connector/I2C_ADDR.2
- J1 pad A6: unconnected-(J1-PadA6) -> /Interboard_connector/UART.TX
- J1 pad A7: unconnected-(J1-PadA7) -> /Interboard_connector/UART.RX
- J1 pad A8: unconnected-(J1-PadA8) -> /Interboard_connector/UART_ADDR.0
- J1 pad A9: unconnected-(J1-PadA9) -> /Interboard_connector/UART_ADDR.1
- J1 pad C1: unconnected-(J1-PadC1) -> /Interboard_connector/Alt_mode.1
- J1 pad C10: unconnected-(J1-PadC10) -> /Interboard_connector/Alt_mode.10
- J1 pad C11: unconnected-(J1-PadC11) -> /Interboard_connector/Alt_mode.11
- J1 pad C12: unconnected-(J1-PadC12) -> /Interboard_connector/Alt_mode.12
- J1 pad C13: unconnected-(J1-PadC13) -> /Interboard_connector/Alt_mode.13
- J1 pad C14: unconnected-(J1-PadC14) -> /Interboard_connector/Alt_mode.14
- J1 pad C15: unconnected-(J1-PadC15) -> /Interboard_connector/Alt_mode.15
- J1 pad C16: unconnected-(J1-PadC16) -> /Interboard_connector/Alt_mode.16
- J1 pad C2: unconnected-(J1-PadC2) -> /Interboard_connector/Alt_mode.2
- J1 pad C3: unconnected-(J1-PadC3) -> /Interboard_connector/Alt_mode.3
- J1 pad C4: unconnected-(J1-PadC4) -> /Interboard_connector/Alt_mode.4
- J1 pad C5: unconnected-(J1-PadC5) -> /Interboard_connector/Alt_mode.5
- J1 pad C6: unconnected-(J1-PadC6) -> /Interboard_connector/Alt_mode.6
- J1 pad C7: unconnected-(J1-PadC7) -> /Interboard_connector/Alt_mode.7
- J1 pad C8: unconnected-(J1-PadC8) -> /Interboard_connector/Alt_mode.8
- J1 pad C9: unconnected-(J1-PadC9) -> /Interboard_connector/Alt_mode.9
- J7 pad 1: GND -> GNDPWR
- J7 pad 2: VCC -> BRD_VIN
- JP301 pad 2: /VRM/TPS563201/+3V3_UNPROTEC -> /VRM/TPS563201/VOUT
- L301 pad 1: /VRM/TPS563201/+3V3_UNPROTEC -> /VRM/TPS563201/SW_3V3
- R400 pad 2: Net-(LED300-Pad1) -> unconnected-(R400-Pad2)
- R407 pad 2: Net-(LED300-Pad3) -> unconnected-(R407-Pad2)
- R408 pad 2: Net-(LED301-Pad1) -> unconnected-(R408-Pad2)
- R409 pad 2: Net-(LED301-Pad3) -> unconnected-(R409-Pad2)
- R8 pad 1: /VRM/LMR36520ADDAR/LMR36520ADDAR_VIN -> BRD_VIN
- R8 pad 2: Net-(C1-Pad2) -> /VRM/LMR36520ADDAR/Cap_protec
- R9 pad 1: Net-(C1-Pad2) -> /VRM/LMR36520ADDAR/Cap_protec
- U2 pad 2: /VRM/LMR36520ADDAR/LMR36520ADDAR_VIN -> BRD_VIN
- U2 pad 3: /VRM/LMR36520ADDAR/LMR36520ADDAR_VIN -> BRD_VIN
- U301 pad 2: /VRM/TPS563201/+3V3_UNPROTEC -> /VRM/TPS563201/SW_3V3
Routing:
- net /CAN auto terminator/CAN2.-: track 37.5 -> 114.7 mm, vias 1 -> 2
- net /CAN auto terminator/CAN1.-: track 26.5 -> 98.9 mm, vias 1 -> 2
- net /CAN auto terminator/CAN1.+: track 32.8 -> 100.2 mm, vias 1 -> 2
- net /CAN auto terminator/CAN2.+: track 46.3 -> 112.3 mm, vias 1 -> 3
- net GND: track 1.81 -> 24.3 mm, vias 0 -> 105
- net /VRM/LMR36520ADDAR/LMR36520ADDAR_VOUT: track 8.07 -> 29.8 mm, vias 0 -> 12
- net +3V3: track 14.3 -> 33.0 mm, vias 0 -> 1
- net /MCU/QSPI1.IO2: track 8.80 -> 19.5 mm
- net Net-(C46-Pad1): track 9.59 -> 1.21 mm
- net Net-(C45-Pad1): track 0.00 -> 6.06 mm
- net /MMS_CONNECTOR_DOWNSTREAM/USB_MMS_CONN.D-: track 74.8 -> 80.5 mm
- net VBUS: track 6.53 -> 12.1 mm
- net /MCU/OSC32_IN: track 0.00 -> 5.53 mm
- net /MCU/OSC32_OUT: track 0.00 -> 5.45 mm
- net /MCU/VDDA: track 0.00 -> 4.59 mm
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- added copper zone on F.Cu, net /VRM/LMR36520ADDAR/Cap_protec
- added copper zone on F.Cu, net /VRM/LMR36520ADDAR/LMR36520ADDAR_VOUT
- added copper zone on F.Cu, net /VRM/TPS563201/+3V3_UNPROTEC
- added copper zone on F.Cu, net /VRM/TPS563201/SW_3V3
- added copper zone on F.Cu, net BRD_VIN
- added copper zone on F.Cu, net GND
Other:
- board text added: "1200W 60V 60A"
- board text added: "21.5khz pi filter or check on vesc forum"
- board text added: "CHAINBUS"
- board text added: "DIN41612"
- board text added: "DOWNLINK"
- board text added: "Encloshure is supposed to have 2mm walls :)"
- board text added: "IEC 60664-1 Material Group III (CTI < 400; typical FR-4 = IIIa): 1.25 mm"
- board text added: "MMS LINK"
- board text added: "Master link"
- board text added: "UPLINK"
- board text added: "USB"
- board text added: "VIN"
- board text added: "VOUT"
