File: PCB-source/MMS2.kicad_sch (KiCad schematic)
At the start: 0 parts

Commit message: vrm VIP
Other:
- sheet CAN terminator renamed CAN auto terminator
- sheet CAN auto terminator ports: added CAN_AUTOTERM{1,2}; removed none

Commit message: Finish component and diffpair placement
Other:
- removed sheet User area
- added sheet Interboard_connector (Interboard_connector.kicad_sch)
- sheet MCU ports: added CAN_AUTOTERM{1,2}; removed none
- note removed: "USER PROJECT"

Commit message: pinout start
Parts:
- added H1, H2, H3, H4: M3 mount, MountingHole:MountingHole_3.2mm_M3_DIN965_Pad, symbol Mechanical:MountingHole_Pad
Connections:
- new net GND: H1.1
- no-connect marks 0 -> 3

Commit message: in progress
Other:
- removed sheet POWER_CONN_IN
- added sheet POWER_IN_CONN (POWER_IN_CONN.kicad_sch)
- moved on the sheet: H1, H2, H3, H4
Changed lines of the file:
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@@
 	)
 	(no_connect
-		(at 74.93 180.34)
+		(at 74.93 171.45)
 	)
 	(no_connect
-		(at 62.23 180.34)
+		(at 62.23 171.45)
 	)
 	(no_connect
-		(at 50.8 180.34)
+		(at 50.8 171.45)
 	)
 	(polyline
@@
 	(wire
 		(pts
-			(xy 35.56 180.34) (xy 35.56 184.15)
+			(xy 35.56 171.45) (xy 35.56 175.26)
 		)
 		(stroke
@@
 	)
 	(image
-		(at 39.37 143.51)
+		(at 41.91 142.24)
 		(scale 0.449816)
 		(data "iVBORw0KGgoAAAANSUhEUgAAAkEAAAGxCAYAAABlfmIpAAAABHNCSVQICAgIfAhkiAAAIABJREFU"
@@
 	(symbol
 		(lib_id "Mechanical:MountingHole_Pad")
-		(at 49.53 177.8 0)
+		(at 49.53 168.91 0)
 		(unit 1)
 		(exclude_from_sim yes)
@@
 		(fields_autoplaced yes)
 		(property "Reference" "H2"
-			(at 52.07 175.26 0)
+			(at 52.07 166.37 0)
 			(effects
 				(font
@@
 		)
 		(property "Value" "M3 mount"
-			(at 52.07 177.8 0)
+			(at 52.07 168.91 0)
 			(effects
 				(font
@@
 		)
 		(property "Footprint" "MountingHole:MountingHole_3.2mm_M3_DIN965_Pad"
-			(at 49.53 177.8 0)
+			(at 49.53 168.91 0)
 			(effects
 				(font
@@
 		)
 		(property "Datasheet" "~"
-			(at 49.53 177.8 0)
+			(at 49.53 168.91 0)
 			(effects
 				(font
@@
 		)
 		(property "Description" "Mounting Hole with connection"
-			(at 49.53 177.8 0)
+			(at 49.53 168.91 0)
 			(effects
 				(font
@@
 	(symbol
 		(lib_id "power:GND")
-		(at 35.56 184.15 0)
+		(at 35.56 175.26 0)
 		(unit 1)
 		(exclude_from_sim no)
@@
 		(fields_autoplaced yes)
 		(property "Reference" "#PWR0101"
-			(at 35.56 190.5 0)
+			(at 35.56 181.61 0)
 			(effects
 				(font
@@
 		)
 		(property "Value" "GND"
-			(at 35.56 189.23 0)
+			(at 35.56 180.34 0)
 			(effects
 				(font
@@
 		)
 		(property "Footprint" ""
-			(at 35.56 184.15 0)
+			(at 35.56 175.26 0)
 			(effects
 				(font
@@
 		)
 		(property "Datasheet" ""
-			(at 35.56 184.15 0)
+			(at 35.56 175.26 0)
 			(effects
 				(font
@@
 		)
 		(property "Description" "Power symbol creates a global label with name \"GND\" , ground"
-			(at 35.56 184.15 0)
+			(at 35.56 175.26 0)
 			(effects
 				(font
@@
 	(symbol
 		(lib_id "Mechanical:MountingHole_Pad")
-		(at 35.56 177.8 0)
+		(at 35.56 168.91 0)
 		(unit 1)
 		(exclude_from_sim yes)
@@
 		(fields_autoplaced yes)
 		(property "Reference" "H1"
-			(at 38.1 175.26 0)
+			(at 38.1 166.37 0)
 			(effects
 				(font
@@
 		)
 		(property "Value" "M3 mount"
-			(at 38.1 177.8 0)
+			(at 38.1 168.91 0)
 			(effects
 				(font
@@
 		)
 		(property "Footprint" "MountingHole:MountingHole_3.2mm_M3_DIN965_Pad"
-			(at 35.56 177.8 0)
+			(at 35.56 168.91 0)
 			(effects
 				(font
@@
 		)
 		(property "Datasheet" "~"
-			(at 35.56 177.8 0)
+			(at 35.56 168.91 0)
 			(effects
 				(font
@@
 		)
 		(property "Description" "Mounting Hole with connection"
-			(at 35.56 177.8 0)
+			(at 35.56 168.91 0)
 			(effects
 				(font
@@
 	(symbol
 		(lib_id "Mechanical:MountingHole_Pad")
-		(at 62.23 177.8 0)
+		(at 62.23 168.91 0)
 		(unit 1)
 		(exclude_from_sim yes)
@@
 		(fields_autoplaced yes)
 		(property "Reference" "H3"
-			(at 64.77 175.26 0)
+			(at 64.77 166.37 0)
 			(effects
 				(font
@@
 		)
 		(property "Value" "M3 mount"
-			(at 64.77 177.8 0)
+			(at 64.77 168.91 0)
 			(effects
 				(font
@@
 		)
 		(property "Footprint" "MountingHole:MountingHole_3.2mm_M3_DIN965_Pad"
-			(at 62.23 177.8 0)
+			(at 62.23 168.91 0)
 			(effects
 				(font
@@
 		)
 		(property "Datasheet" "~"
-			(at 62.23 177.8 0)
+			(at 62.23 168.91 0)
 			(effects
 				(font
@@
 		)
 		(property "Description" "Mounting Hole with connection"
-			(at 62.23 177.8 0)
+			(at 62.23 168.91 0)
 			(effects
 				(font
@@
 	(symbol
 		(lib_id "Mechanical:MountingHole_Pad")
-		(at 74.93 177.8 0)
+		(at 74.93 168.91 0)
 		(unit 1)
 		(exclude_from_sim yes)
@@
 		(fields_autoplaced yes)
 		(property "Reference" "H4"
-			(at 77.47 175.26 0)
+			(at 77.47 166.37 0)
 			(effects
 				(font
@@
 		)
 		(property "Value" "M3 mount"
-			(at 77.47 177.8 0)
+			(at 77.47 168.91 0)
 			(effects
 				(font
@@
 		)
 		(property "Footprint" "MountingHole:MountingHole_3.2mm_M3_DIN965_Pad"
-			(at 74.93 177.8 0)
+			(at 74.93 168.91 0)
 			(effects
 				(font
@@
 		)
 		(property "Datasheet" "~"
-			(at 74.93 177.8 0)
+			(at 74.93 168.91 0)
 			(effects
 				(font
@@
 		)
 		(property "Description" "Mounting Hole with connection"
-			(at 74.93 177.8 0)
+			(at 74.93 168.91 0)
 			(effects
 				(font
@@
 	)
 	(sheet
+		(at 25.4 129.54)
+		(size 30.48 24.13)
+		(exclude_from_sim no)
+		(in_bom yes)
+		(on_board yes)
+		(dnp no)
+		(fields_autoplaced yes)
+		(stroke
+			(width 0.1524)
+			(type solid)
+		)
+		(fill
+			(color 0 0 0 0.0000)
+		)
+		(property "Sheetname" "POWER_IN_CONN"
+			(at 25.4 128.8284 0)
+			(effects
+				(font
+					(size 1.27 1.27)
+				)
+				(justify left bottom)
+			)
+		)
+		(property "Sheetfile" "POWER_IN_CONN.kicad_sch"
+			(at 25.4 154.2546 0)
+			(effects
+				(font
+					(size 1.27 1.27)
+				)
+				(justify left top)
+			)
+		)
+		(instances
+			(project "MMS2"
+				(path "/6596548a-44e0-46d8-8624-fd71cf4a3e17"
+					(page "20")
+				)
+			)
+		)
+	)
+	(sheet
 		(at 67.31 99.06)
 		(size 44.45 8.89)
@@
 				)
 			)
-		)
-	)
-	(sheet
-		(at 24.13 129.54)
-		(size 31.75 26.67)
-		(exclude_from_sim no)
-		(in_bom yes)
-		(on_board yes)
-		(dnp no)
-		(fields_autoplaced yes)
-		(stroke
-			(width 0.1524)
-			(type solid)
-		)
-		(fill
-			(color 0 0 0 0.0000)
-		)
-		(property "Sheetname" "POWER_CONN_IN"
-			(at 24.13 128.8284 0)
-			(effects
-				(font
-					(size 1.27 1.27)
-				)
-				(justify left bottom)
-			)
-		)
-		(property "Sheetfile" "POWER_CONN.kicad_sch"
-			(at 24.13 156.7946 0)
-			(effects
-				(font
-					(size 1.27 1.27)
-				)
-				(justify left top)
-			)
-		)
-		(instances
-			(project "MMS2"
-				(path "/6596548a-44e0-46d8-8624-fd71cf4a3e17"
-					(page "15")
-				)
-			)
