File: PCB-source/POWER_IN_CONN.kicad_sch (KiCad schematic)
At the start: 1 part, among them J7 AMASS XT60

Commit message: in progress
Parts:
- removed J7: AMASS XT60, XT60:AMASS_XT60PW-F_1x02_P7.20mm_Horizontal, symbol Connector_Generic:Conn_01x02
- added J2: AMASS XT60, XT60:AMASS_XT60PW-M_1x02_P7.20mm_Horizontal, symbol Connector_Generic:Conn_01x02
Connections:
- net BRD_VIN: now also J2.2 (Pin_2)
- net GNDPWR: now also J2.1 (Pin_1)
Other:
- company: Moducard System -> (none)
- title: MMS2 -> (none)
Changed lines of the file:
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@@
 	(generator_version "9.0")
 	(paper "A4")
-	(title_block
-		(title "MMS2")
-		(date "2025-04-22")
-		(rev "A")
-		(company "Moducard System")
-		(comment 1 "Artem Horiunov")
-		(comment 2 "Designed in poland")
-	)
-	(wire
-		(pts
-			(xy 137.16 95.25) (xy 133.35 95.25)
-		)
-		(stroke
-			(width 0)
-			(type default)
-		)
-	)
-	(wire
-		(pts
-			(xy 137.16 92.71) (xy 137.16 95.25)
-		)
-		(stroke
-			(width 0)
-			(type default)
-		)
-	)
-	(wire
-		(pts
-			(xy 137.16 97.79) (xy 137.16 100.33)
-		)
-		(stroke
-			(width 0)
-			(type default)
-		)
-	)
-	(wire
-		(pts
-			(xy 133.35 97.79) (xy 137.16 97.79)
+	(wire
+		(pts
+			(xy 143.51 97.79) (xy 139.7 97.79)
+		)
+		(stroke
+			(width 0)
+			(type default)
+		)
+	)
+	(wire
+		(pts
+			(xy 139.7 100.33) (xy 143.51 100.33)
+		)
+		(stroke
+			(width 0)
+			(type default)
+		)
+	)
+	(wire
+		(pts
+			(xy 143.51 95.25) (xy 143.51 97.79)
+		)
+		(stroke
+			(width 0)
+			(type default)
+		)
+	)
+	(wire
+		(pts
+			(xy 143.51 100.33) (xy 143.51 102.87)
 		)
 		(stroke
@@
 	(symbol
 		(lib_id "Connector_Generic:Conn_01x02")
-		(at 128.27 97.79 180)
+		(at 134.62 100.33 180)
 		(unit 1)
 		(exclude_from_sim no)
@@
 		(dnp no)
 		(fields_autoplaced yes)
-		(property "Reference" "J7"
-			(at 128.27 88.9 0)
+		(property "Reference" "J2"
+			(at 134.62 91.44 0)
 			(effects
 				(font
@@
 		)
 		(property "Value" "AMASS XT60"
-			(at 128.27 91.44 0)
-			(effects
-				(font
-					(size 1.27 1.27)
-				)
-			)
-		)
-		(property "Footprint" "XT60:AMASS_XT60PW-F_1x02_P7.20mm_Horizontal"
-			(at 128.27 97.79 0)
+			(at 134.62 93.98 0)
+			(effects
+				(font
+					(size 1.27 1.27)
+				)
+			)
+		)
+		(property "Footprint" "XT60:AMASS_XT60PW-M_1x02_P7.20mm_Horizontal"
+			(at 134.62 100.33 0)
 			(effects
 				(font
@@
 		)
 		(property "Datasheet" "~"
-			(at 128.27 97.79 0)
+			(at 134.62 100.33 0)
 			(effects
 				(font
@@
 		)
 		(property "Description" "Generic connector, single row, 01x02, script generated (kicad-library-utils/schlib/autogen/connector/)"
-			(at 128.27 97.79 0)
+			(at 134.62 100.33 0)
 			(effects
 				(font
@@
 		(instances
 			(project "MMS2"
-				(path "/6596548a-44e0-46d8-8624-fd71cf4a3e17/90d9dcde-6a4d-4313-9bcc-0dca5a9ec8a8"
-					(reference "J7")
+				(path "/6596548a-44e0-46d8-8624-fd71cf4a3e17/75744aa8-9b7c-4f01-8c3f-b5153be45f3f"
+					(reference "J2")
 					(unit 1)
 				)
@@
 	(symbol
 		(lib_id "power:VCC")
-		(at 137.16 92.71 0)
+		(at 143.51 95.25 0)
 		(unit 1)
 		(exclude_from_sim no)
@@
 		(dnp no)
 		(fields_autoplaced yes)
-		(property "Reference" "#PWR023"
-			(at 137.16 96.52 0)
+		(property "Reference" "#PWR022"
+			(at 143.51 99.06 0)
 			(effects
 				(font
@@
 		)
 		(property "Value" "BRD_VIN"
-			(at 137.16 87.63 0)
+			(at 143.51 90.17 0)
 			(effects
 				(font
@@
 		)
 		(property "Footprint" ""
-			(at 137.16 92.71 0)
+			(at 143.51 95.25 0)
 			(effects
 				(font
@@
 		)
 		(property "Datasheet" ""
-			(at 137.16 92.71 0)
+			(at 143.51 95.25 0)
 			(effects
 				(font
@@
 		)
 		(property "Description" "Power symbol creates a global label with name \"VCC\""
-			(at 137.16 92.71 0)
+			(at 143.51 95.25 0)
 			(effects
 				(font
@@
 		)
 		(instances
-			(project "MMS2"
-				(path "/6596548a-44e0-46d8-8624-fd71cf4a3e17/90d9dcde-6a4d-4313-9bcc-0dca5a9ec8a8"
-					(reference "#PWR023")
+			(project ""
+				(path "/6596548a-44e0-46d8-8624-fd71cf4a3e17/75744aa8-9b7c-4f01-8c3f-b5153be45f3f"
+					(reference "#PWR022")
 					(unit 1)
 				)
@@
 	(symbol
 		(lib_id "power:GNDPWR")
-		(at 137.16 100.33 0)
+		(at 143.51 102.87 0)
 		(unit 1)
 		(exclude_from_sim no)
@@
 		(dnp no)
 		(fields_autoplaced yes)
-		(property "Reference" "#PWR025"
-			(at 137.16 105.41 0)
+		(property "Reference" "#PWR024"
+			(at 143.51 107.95 0)
 			(effects
 				(font
@@
 		)
 		(property "Value" "GNDPWR"
-			(at 137.033 104.14 0)
+			(at 143.383 106.68 0)
 			(effects
 				(font
@@
 		)
 		(property "Footprint" ""
-			(at 137.16 101.6 0)
+			(at 143.51 104.14 0)
 			(effects
 				(font
@@
 		)
 		(property "Datasheet" ""
-			(at 137.16 101.6 0)
+			(at 143.51 104.14 0)
 			(effects
 				(font
@@
 		)
 		(property "Description" "Power symbol creates a global label with name \"GNDPWR\" , global ground"
-			(at 137.16 100.33 0)
+			(at 143.51 102.87 0)
 			(effects
 				(font
@@
 		)
 		(instances
-			(project "MMS2"
-				(path "/6596548a-44e0-46d8-8624-fd71cf4a3e17/90d9dcde-6a4d-4313-9bcc-0dca5a9ec8a8"
-					(reference "#PWR025")
+			(project ""
+				(path "/6596548a-44e0-46d8-8624-fd71cf4a3e17/75744aa8-9b7c-4f01-8c3f-b5153be45f3f"
+					(reference "#PWR024")
 					(unit 1)
 				)
