File: PCB-source/STlink-BMprobe.kicad_sch (KiCad schematic)
At the start: 38 parts, among them Q700 MMST3904, U700 STM32F103CBTx, Y700 Crystal_GND24

Commit message: vrm VIP
Other:
- note added: "Do weryfikackji moducard nav module 2"
- note removed: "Do weryfikackji"
Changed lines of the file:
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@@
 		)
 	)
-	(text "Do weryfikackji"
+	(text "Do weryfikackji moducard nav module 2\n"
 		(exclude_from_sim no)
 		(at 124.46 148.082 0)

Commit message: Finish component and diffpair placement
Parts:
- Q700: footprint PCM_JLCPCB:Q_SOT-323 -> Package_TO_SOT_SMD:SOT-23
Other:
- note added: "Podłączyć do UART1 stmH5"
- title: MMS2 -> Black magic probe
Changed lines of the file:
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@@
 	(paper "A4")
 	(title_block
-		(title "MMS2")
+		(title "Black magic probe")
 		(date "2025-04-22")
 		(rev "A")
@@
 		)
 	)
+	(text "Podłączyć do UART1 stmH5\n"
+		(exclude_from_sim no)
+		(at 189.992 62.484 0)
+		(effects
+			(font
+				(size 5.08 5.08)
+				(thickness 1.016)
+				(bold yes)
+				(color 255 0 93 1)
+			)
+		)
+	)
 	(text "Populate with STM32F103C8, STM32F103CB\n"
 		(exclude_from_sim no)
@@
 	(text "Do weryfikackji moducard nav module 2\n"
 		(exclude_from_sim no)
-		(at 124.46 148.082 0)
+		(at 125.222 157.988 0)
 		(effects
 			(font
@@
 	)
 	(bus_entry
-		(at 127 111.76)
+		(at 135.89 111.76)
 		(size 2.54 2.54)
 		(stroke
@@
 	)
 	(bus_entry
-		(at 127 109.22)
+		(at 135.89 109.22)
 		(size 2.54 2.54)
 		(stroke
@@
 	)
 	(bus_entry
-		(at 127 114.3)
+		(at 135.89 114.3)
 		(size 2.54 2.54)
 		(stroke
@@
 	(wire
 		(pts
-			(xy 114.3 109.22) (xy 127 109.22)
+			(xy 123.19 109.22) (xy 135.89 109.22)
 		)
 		(stroke
@@
 	(bus
 		(pts
-			(xy 129.54 119.38) (xy 130.81 120.65)
+			(xy 138.43 119.38) (xy 139.7 120.65)
 		)
 		(stroke
@@
 	(bus
 		(pts
-			(xy 130.81 120.65) (xy 133.35 120.65)
+			(xy 139.7 120.65) (xy 142.24 120.65)
 		)
 		(stroke
@@
 		)
 	)
+	(polyline
+		(pts
+			(xy 153.67 67.31) (xy 137.16 68.58)
+		)
+		(stroke
+			(width 0)
+			(type default)
+		)
+	)
 	(wire
 		(pts
@@
 	(bus
 		(pts
-			(xy 129.54 116.84) (xy 129.54 119.38)
+			(xy 138.43 116.84) (xy 138.43 119.38)
 		)
 		(stroke
@@
 	(wire
 		(pts
-			(xy 114.3 114.3) (xy 127 114.3)
+			(xy 123.19 114.3) (xy 135.89 114.3)
 		)
 		(stroke
@@
 	(bus
 		(pts
-			(xy 129.54 114.3) (xy 129.54 116.84)
+			(xy 138.43 114.3) (xy 138.43 116.84)
 		)
 		(stroke
@@
 	(wire
 		(pts
-			(xy 114.3 111.76) (xy 127 111.76)
+			(xy 123.19 111.76) (xy 135.89 111.76)
 		)
 		(stroke
@@
 		)
 	)
+	(polyline
+		(pts
+			(xy 137.16 68.58) (xy 138.43 69.85)
+		)
+		(stroke
+			(width 0)
+			(type default)
+		)
+	)
 	(wire
 		(pts
@@
 		)
 	)
+	(polyline
+		(pts
+			(xy 137.16 68.58) (xy 138.43 67.31)
+		)
+		(stroke
+			(width 0)
+			(type default)
+		)
+	)
 	(wire
 		(pts
@@
 	(bus
 		(pts
-			(xy 129.54 114.3) (xy 129.54 111.76)
+			(xy 138.43 114.3) (xy 138.43 111.76)
 		)
 		(stroke
@@
 	)
 	(label "SWD.SWCLK"
-		(at 114.3 111.76 0)
+		(at 123.19 111.76 0)
 		(effects
 			(font
@@
 	)
 	(label "SWD.SWDIO"
-		(at 114.3 109.22 0)
+		(at 123.19 109.22 0)
 		(effects
 			(font
@@
 	)
 	(label "SWD.~{RST}"
-		(at 114.3 114.3 0)
+		(at 123.19 114.3 0)
 		(effects
 			(font
@@
 	(hierarchical_label "SWD{SWD}"
 		(shape output)
-		(at 133.35 120.65 0)
+		(at 142.24 120.65 0)
 		(effects
 			(font
@@
 		(on_board yes)
 		(dnp no)
-		(fields_autoplaced yes)
 		(property "Reference" "U700"
-			(at 103.7941 133.35 0)
+			(at 103.124 135.128 0)
 			(effects
 				(font
@@
 		)
 		(property "Value" "STM32F103CBTx"
-			(at 103.7941 135.89 0)
+			(at 103.124 137.668 0)
 			(effects
 				(font
@@
 			)
 		)
-		(property "Footprint" "PCM_JLCPCB:Q_SOT-323"
+		(property "Footprint" "Package_TO_SOT_SMD:SOT-23"
 			(at 236.728 96.52 90)
 			(effects

Commit message: in progress
Changed lines of the file:
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@@
 	(text "Podłączyć do UART1 stmH5\n"
 		(exclude_from_sim no)
-		(at 189.992 62.484 0)
+		(at 206.248 62.484 0)
 		(effects
 			(font
@@
 	(polyline
 		(pts
-			(xy 153.67 67.31) (xy 137.16 68.58)
+			(xy 154.94 67.31) (xy 138.43 68.58)
 		)
 		(stroke
@@
 	(polyline
 		(pts
-			(xy 137.16 68.58) (xy 138.43 69.85)
+			(xy 138.43 68.58) (xy 139.7 69.85)
 		)
 		(stroke
@@
 	(polyline
 		(pts
-			(xy 137.16 68.58) (xy 138.43 67.31)
-		)
-		(stroke
+			(xy 138.43 68.58) (xy 139.7 67.31)
+		)
+		(stroke
